File: board/board.kicad_sch (KiCad schematic)
At the start: 38 parts, among them U101 Pico, U102 CS42438

Commit message: pcb done
attempt at doing some sw. builds but not tested
Connections:
- net GNDA: now also H101.1, H102.1, H103.1
- net GNDD: now also H104.1
- net dac_aux_lrck: now also U101.12 (GPIO9); no longer U101.25 (GPIO19)
- net dac_aux_sclk: now also U101.11 (GPIO8); no longer U101.26 (GPIO20)
- net dac_aux_sdin: now also U101.10 (GPIO7); no longer U101.27 (GPIO21)
- net dac_ctrl_cipo: now also U101.21 (GPIO16); no longer U101.16 (GPIO12)
- net dac_ctrl_clk: now also U101.24 (GPIO18); no longer U101.19 (GPIO14)
- net dac_ctrl_copi: now also U101.25 (GPIO19); no longer U101.20 (GPIO15)
- net dac_ctrl_csn: now also U101.22 (GPIO17); no longer U101.17 (GPIO13)
- net dac_ctrl_rstn: now also R106.1, U101.26 (GPIO20); no longer U101.15 (GPIO11)
- net dac_ctrl_rstn_term: no longer R106.1
- net dac_fs: now also U101.15 (GPIO11); no longer U101.12 (GPIO9)
- net dac_mclk: now also U101.20 (GPIO15); no longer U101.14 (GPIO10)
- net dac_sclk: now also U101.16 (GPIO12); no longer U101.11 (GPIO8)
- net dac_sdin: now also U101.19 (GPIO14); no longer U101.9 (GPIO6)
- net dac_sdout: now also U101.17 (GPIO13); no longer U101.10 (GPIO7)
- net transz_rf3: now reaches U101.1 (GPIO0)
- net transz_rf2: now reaches U101.2 (GPIO1)
- net transz_rf1: now reaches U101.4 (GPIO2)
- removed net GNDPWR: H101.1, H102.1, H103.1, H104.1
- no-connect marks 22 -> 39
Other:
- moved on the sheet: C111, C114, D101, FB101, H101, H102, H103, H104, R106, U101

Commit message: Order pcb
Connections:
- net GNDA: no longer H103.1
- net GNDD: now also H103.1
Changed lines of the file:
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@@
   (junction (at 193.675 37.465) (diameter 0) (color 0 0 0 0)
   )
-  (junction (at 216.535 37.465) (diameter 0) (color 0 0 0 0)
-  )
   (junction (at 122.555 126.365) (diameter 0) (color 0 0 0 0)
   )
@@
   )
   (junction (at 126.365 106.68) (diameter 0) (color 0 0 0 0)
+  )
+  (junction (at 260.985 37.465) (diameter 0) (color 0 0 0 0)
   )
   (junction (at 64.135 59.055) (diameter 0) (color 0 0 0 0)
@@
     (stroke (width 0) (type default) (color 0 0 0 0))
   )
-  (bus_entry (at 53.34 28.575) (size 2.54 2.54)
-    (stroke (width 0) (type default) (color 0 0 0 0))
-  )
-  (bus_entry (at 53.34 26.035) (size 2.54 2.54)
-    (stroke (width 0) (type default) (color 0 0 0 0))
-  )
-  (bus_entry (at 53.34 33.655) (size 2.54 2.54)
+  (bus_entry (at 50.8 28.575) (size 2.54 2.54)
+    (stroke (width 0) (type default) (color 0 0 0 0))
+  )
+  (bus_entry (at 50.8 26.035) (size 2.54 2.54)
+    (stroke (width 0) (type default) (color 0 0 0 0))
+  )
+  (bus_entry (at 50.8 33.655) (size 2.54 2.54)
     (stroke (width 0) (type default) (color 0 0 0 0))
   )
@@
     (stroke (width 0) (type default) (color 0 0 0 0))
   )
-  (bus (pts (xy 53.34 26.035) (xy 53.34 28.575))
+  (bus (pts (xy 50.8 26.035) (xy 50.8 28.575))
     (stroke (width 0) (type default) (color 0 0 0 0))
   )
@@
     (stroke (width 0) (type default) (color 0 0 0 0))
   )
-  (wire (pts (xy 55.88 31.115) (xy 66.675 31.115))
+  (wire (pts (xy 53.34 31.115) (xy 66.675 31.115))
     (stroke (width 0) (type default) (color 0 0 0 0))
   )
@@
     (stroke (width 0) (type default) (color 0 0 0 0))
   )
-  (bus (pts (xy 53.34 28.575) (xy 53.34 33.655))
+  (bus (pts (xy 50.8 28.575) (xy 50.8 33.655))
     (stroke (width 0) (type default) (color 0 0 0 0))
   )
@@
     (stroke (width 0) (type default) (color 0 0 0 0))
   )
-  (bus (pts (xy 53.34 20.32) (xy 53.34 26.035))
+  (bus (pts (xy 50.8 20.32) (xy 50.8 26.035))
     (stroke (width 0) (type default) (color 0 0 0 0))
   )
@@
     (stroke (width 0) (type default) (color 0 0 0 0))
   )
-  (wire (pts (xy 238.76 37.465) (xy 216.535 37.465))
+  (wire (pts (xy 260.985 38.735) (xy 260.985 37.465))
     (stroke (width 0) (type default) (color 0 0 0 0))
   )
@@
     (stroke (width 0) (type default) (color 0 0 0 0))
   )
-  (wire (pts (xy 55.88 28.575) (xy 66.675 28.575))
+  (wire (pts (xy 53.34 28.575) (xy 66.675 28.575))
     (stroke (width 0) (type default) (color 0 0 0 0))
   )
@@
     (stroke (width 0) (type default) (color 0 0 0 0))
   )
+  (wire (pts (xy 64.135 33.655) (xy 64.135 46.355))
+    (stroke (width 0) (type default) (color 0 0 0 0))
+  )
   (wire (pts (xy 161.29 57.15) (xy 168.275 57.15))
     (stroke (width 0) (type default) (color 0 0 0 0))
@@
     (stroke (width 0) (type default) (color 0 0 0 0))
   )
-  (wire (pts (xy 55.88 36.195) (xy 66.675 36.195))
+  (wire (pts (xy 53.34 36.195) (xy 66.675 36.195))
     (stroke (width 0) (type default) (color 0 0 0 0))
   )
@@
     (stroke (width 0) (type default) (color 0 0 0 0))
   )
+  (wire (pts (xy 238.76 37.465) (xy 260.985 37.465))
+    (stroke (width 0) (type default) (color 0 0 0 0))
+  )
   (wire (pts (xy 66.675 71.755) (xy 64.135 71.755))
     (stroke (width 0) (type default) (color 0 0 0 0))
@@
     (stroke (width 0) (type default) (color 0 0 0 0))
   )
-  (bus (pts (xy 53.34 20.32) (xy 131.445 20.32))
+  (bus (pts (xy 50.8 20.32) (xy 131.445 20.32))
     (stroke (width 0) (type default) (color 0 0 0 0))
   )
@@
   )
   (wire (pts (xy 229.87 140.335) (xy 229.87 116.205))
-    (stroke (width 0) (type default) (color 0 0 0 0))
-  )
-  (wire (pts (xy 64.135 33.655) (xy 64.135 46.355))
     (stroke (width 0) (type default) (color 0 0 0 0))
   )
@@
     (effects (font (size 1.27 1.27)) (justify left bottom))
   )
-  (label "transz_rf2" (at 56.515 31.115 0)
+  (label "transz_rf2" (at 53.975 31.115 0)
     (effects (font (size 1.27 1.27)) (justify left bottom))
   )
@@
     (effects (font (size 1.27 1.27)) (justify left bottom))
   )
-  (label "transz_rf1" (at 56.515 36.195 0)
+  (label "transz_rf1" (at 53.975 36.195 0)
     (effects (font (size 1.27 1.27)) (justify left bottom))
   )
@@
     (effects (font (size 1.27 1.27)) (justify left bottom))
   )
-  (label "transz_rf3" (at 56.515 28.575 0)
+  (label "transz_rf3" (at 53.975 28.575 0)
     (effects (font (size 1.27 1.27)) (justify left bottom))
   )
@@
     (pin "2")
   )
-  (symbol (lib_id "power:GNDD") (at 260.985 37.465 0) (unit 1)
-    (in_bom yes) (on_board yes) (fields_autoplaced)
-    (property "Reference" "#PWR0131" (id 0) (at 260.985 43.815 0)
-      (effects (font (size 1.27 1.27)) hide)
-    )
-    (property "Value" "GNDD" (id 1) (at 260.985 41.6465 0))
-    (property "Footprint" "" (id 2) (at 260.985 37.465 0)
-      (effects (font (size 1.27 1.27)) hide)
-    )
-    (property "Datasheet" "" (id 3) (at 260.985 37.465 0)
-      (effects (font (size 1.27 1.27)) hide)
-    )
+  (symbol (lib_id "power:GNDD") (at 260.985 38.735 0) (unit 1)
+    (in_bom yes) (on_board yes) (fields_autoplaced)
+    (property "Reference" "#PWR0131" (id 0) (at 260.985 45.085 0)
+      (effects (font (size 1.27 1.27)) hide)
+    )
+    (property "Value" "GNDD" (id 1) (at 260.985 42.9165 0))
+    (property "Footprint" "" (id 2) (at 260.985 38.735 0)
+      (effects (font (size 1.27 1.27)) hide)
+    )
+    (property "Datasheet" "" (id 3) (at 260.985 38.735 0)
+      (effects (font (size 1.27 1.27)) hide)
+    )

Commit message: stuff
Parts:
- U102: footprint Package_QFP:LQFP-52_10x10mm_P0.65mm -> good_things:QFP-52_14x14_Pitch0.65mm
Changed lines of the file:
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@@
     (property "Reference" "U102" (id 0) (at 191.135 48.1543 0))
     (property "Value" "CS42438" (id 1) (at 191.135 50.9294 0))
-    (property "Footprint" "Package_QFP:LQFP-52_10x10mm_P0.65mm" (id 2) (at 192.405 45.085 0)
+    (property "Footprint" "good_things:QFP-52_14x14_Pitch0.65mm" (id 2) (at 192.405 45.085 0)
       (effects (font (size 1.27 1.27)) hide)
     )
@@
     )
     (path "/f7cf94e2-d350-43e4-87cd-d57203670d81"
-      (reference "U102") (unit 1) (value "CS42438") (footprint "Package_QFP:LQFP-52_10x10mm_P0.65mm")
+      (reference "U102") (unit 1) (value "CS42438") (footprint "good_things:QFP-52_14x14_Pitch0.65mm")
     )
     (path "/7b9c2940-9a15-4fc8-9338-3451987ef45d/53526f67-42ef-48a6-b2d6-d8938fc945f8"
