File: board/output_stage.kicad_sch (KiCad schematic)
At the start: 23 parts, among them J301 Conn_Coaxial, U301 lmc6042

Commit message: Some more layout, digital side has been reorganized
looking into single to diff conversion. with the biases
Parts:
- renumbered C301 to C401, C302 to C402, C303 to C403, C304 to C404, C305 to C405, C306 to C406, C307 to C407, C308 to C408, FB301 to FB401, J301 to J401, R301 to R401, R302 to R402, R303 to R403, R304 to R404, R305 to R405, R306 to R406, R307 to R407, R308 to R408, R309 to R409, R310 to R410, U301 to U401
Changed lines of the file:
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@@
   (symbol (lib_id "Device:C_Small") (at 43.18 170.18 0)
     (in_bom yes) (on_board yes)
-    (property "Reference" "C301" (id 0) (at 45.72 169.545 0)
+    (property "Reference" "C401" (id 0) (at 45.72 169.545 0)
       (effects (font (size 1.27 1.27)) (justify left))
     )
@@
   (symbol (lib_id "Device:R") (at 44.45 94.615 90)
     (in_bom yes) (on_board yes)
-    (property "Reference" "R302" (id 0) (at 38.735 93.345 90))
+    (property "Reference" "R402" (id 0) (at 38.735 93.345 90))
     (property "Value" "5k49" (id 1) (at 50.165 93.345 90))
     (property "Footprint" "Resistor_SMD:R_0603_1608Metric_Pad0.98x0.95mm_HandSolder" (id 2) (at 44.45 96.393 90)
@@
   (symbol (lib_id "Device:C_Small") (at 130.81 106.045 270)
     (in_bom yes) (on_board yes) (fields_autoplaced)
-    (property "Reference" "C307" (id 0) (at 130.8036 100.5164 90))
+    (property "Reference" "C407" (id 0) (at 130.8036 100.5164 90))
     (property "Value" "390p" (id 1) (at 130.8036 103.2915 90))
     (property "Footprint" "Capacitor_SMD:C_0603_1608Metric_Pad1.08x0.95mm_HandSolder" (id 2) (at 130.81 106.045 0)
@@
   (symbol (lib_id "Device:Opamp_Dual") (at 209.55 94.615 0)
     (in_bom yes) (on_board yes) (fields_autoplaced)
-    (property "Reference" "U301" (id 0) (at 209.55 85.5685 0))
+    (property "Reference" "U401" (id 0) (at 209.55 85.5685 0))
     (property "Value" "lmc6042" (id 1) (at 209.55 88.3436 0))
     (property "Footprint" "Package_SO:SOIC-8_3.9x4.9mm_P1.27mm" (id 2) (at 209.55 94.615 0)
@@
       (effects (font (size 1.27 1.27)) hide)
     )
-    (pin "5")
-    (pin "6")
-    (pin "7")
+    (pin "1")
+    (pin "2")
+    (pin "3")
   )
   (symbol (lib_id "Connector:Conn_Coaxial") (at 268.605 94.615 0)
     (in_bom yes) (on_board yes) (fields_autoplaced)
-    (property "Reference" "J301" (id 0) (at 271.145 93.9997 0)
+    (property "Reference" "J401" (id 0) (at 271.145 93.9997 0)
       (effects (font (size 1.27 1.27)) (justify left))
     )
@@
   (symbol (lib_id "Device:Opamp_Dual") (at 63.5 170.18 0)
     (in_bom yes) (on_board yes)
-    (property "Reference" "U301" (id 0) (at 61.595 169.2715 0)
+    (property "Reference" "U401" (id 0) (at 61.595 169.2715 0)
       (effects (font (size 1.27 1.27)) (justify left))
     )
@@
       (effects (font (size 1.27 1.27)) hide)
     )
-    (pin "4")
-    (pin "8")
+    (pin "1")
+    (pin "2")
+    (pin "3")
   )
   (symbol (lib_id "power:GNDA") (at 60.96 180.34 0)
@@
   (symbol (lib_id "Device:FerriteBead_Small") (at 67.31 161.29 90)
     (in_bom yes) (on_board yes)
-    (property "Reference" "FB301" (id 0) (at 67.2719 155.6217 90))
+    (property "Reference" "FB401" (id 0) (at 67.2719 155.6217 90))
     (property "Value" "BLM18AG102SN1D" (id 1) (at 67.2719 158.3968 90))
     (property "Footprint" "Inductor_SMD:L_0603_1608Metric_Pad1.05x0.95mm_HandSolder" (id 2) (at 67.31 163.068 90)
@@
   (symbol (lib_id "Device:R") (at 98.425 89.535 90)
     (in_bom yes) (on_board yes)
-    (property "Reference" "R304" (id 0) (at 92.71 88.265 90))
+    (property "Reference" "R404" (id 0) (at 92.71 88.265 90))
     (property "Value" "887" (id 1) (at 103.505 88.265 90))
     (property "Footprint" "Resistor_SMD:R_0603_1608Metric_Pad0.98x0.95mm_HandSolder" (id 2) (at 98.425 91.313 90)
@@
   (symbol (lib_id "Device:C_Small") (at 69.85 71.12 0)
     (in_bom yes) (on_board yes) (fields_autoplaced)
-    (property "Reference" "C305" (id 0) (at 72.1741 70.2178 0)
+    (property "Reference" "C405" (id 0) (at 72.1741 70.2178 0)
       (effects (font (size 1.27 1.27)) (justify left))
     )
@@
   (symbol (lib_id "Device:R") (at 166.37 92.075 90)
     (in_bom yes) (on_board yes)
-    (property "Reference" "R307" (id 0) (at 161.29 90.805 90))
+    (property "Reference" "R407" (id 0) (at 161.29 90.805 90))
     (property "Value" "10k" (id 1) (at 171.45 90.805 90))
     (property "Footprint" "Resistor_SMD:R_0603_1608Metric_Pad0.98x0.95mm_HandSolder" (id 2) (at 166.37 93.853 90)
@@
   (symbol (lib_id "Device:R") (at 245.11 94.615 90)
     (in_bom yes) (on_board yes)
-    (property "Reference" "R310" (id 0) (at 248.92 93.345 90))
+    (property "Reference" "R410" (id 0) (at 248.92 93.345 90))
     (property "Value" "33" (id 1) (at 240.665 93.345 90))
     (property "Footprint" "Resistor_SMD:R_0603_1608Metric_Pad0.98x0.95mm_HandSolder" (id 2) (at 245.11 96.393 90)
@@
   (symbol (lib_id "Device:C_Small") (at 116.84 81.915 0)
     (in_bom yes) (on_board yes) (fields_autoplaced)
-    (property "Reference" "C306" (id 0) (at 119.1641 81.0128 0)
+    (property "Reference" "C406" (id 0) (at 119.1641 81.0128 0)
       (effects (font (size 1.27 1.27)) (justify left))
     )
@@
   (symbol (lib_id "Device:R") (at 98.425 94.615 90)
     (in_bom yes) (on_board yes)
-    (property "Reference" "R305" (id 0) (at 92.71 93.345 90))
+    (property "Reference" "R405" (id 0) (at 92.71 93.345 90))
     (property "Value" "2k94" (id 1) (at 104.14 93.345 90))
     (property "Footprint" "Resistor_SMD:R_0603_1608Metric_Pad0.98x0.95mm_HandSolder" (id 2) (at 98.425 96.393 90)
@@
   (symbol (lib_id "Device:R") (at 130.81 111.125 90)
     (in_bom yes) (on_board yes)
-    (property "Reference" "R306" (id 0) (at 125.095 109.855 90))
+    (property "Reference" "R406" (id 0) (at 125.095 109.855 90))
     (property "Value" "4k75" (id 1) (at 135.89 109.855 90))
     (property "Footprint" "Resistor_SMD:R_0603_1608Metric_Pad0.98x0.95mm_HandSolder" (id 2) (at 130.81 112.903 90)
@@
   (symbol (lib_id "Device:C_Small") (at 61.595 81.915 0)
     (in_bom yes) (on_board yes) (fields_autoplaced)
-    (property "Reference" "C304" (id 0) (at 63.9191 81.0128 0)
+    (property "Reference" "C404" (id 0) (at 63.9191 81.0128 0)
       (effects (font (size 1.27 1.27)) (justify left))
     )
@@
   (symbol (lib_id "Device:R") (at 198.12 113.665 180)
     (in_bom yes) (on_board yes)
-    (property "Reference" "R308" (id 0) (at 196.85 119.38 90))
+    (property "Reference" "R408" (id 0) (at 196.85 119.38 90))
     (property "Value" "10k" (id 1) (at 196.85 109.22 90))
     (property "Footprint" "Resistor_SMD:R_0603_1608Metric_Pad0.98x0.95mm_HandSolder" (id 2) (at 199.898 113.665 90)
@@
   (symbol (lib_id "Device:R") (at 44.45 89.535 90)
     (in_bom yes) (on_board yes)
-    (property "Reference" "R301" (id 0) (at 38.735 88.265 90))
+    (property "Reference" "R401" (id 0) (at 38.735 88.265 90))
     (property "Value" "1k65" (id 1) (at 50.165 88.265 90))
     (property "Footprint" "Resistor_SMD:R_0603_1608Metric_Pad0.98x0.95mm_HandSolder" (id 2) (at 44.45 91.313 90)
@@
   (symbol (lib_id "Device:R") (at 69.85 81.915 180)
     (in_bom yes) (on_board yes)
-    (property "Reference" "R303" (id 0) (at 68.58 86.995 90))
+    (property "Reference" "R403" (id 0) (at 68.58 86.995 90))
     (property "Value" "1k87" (id 1) (at 68.58 76.835 90))
     (property "Footprint" "Resistor_SMD:R_0603_1608Metric_Pad0.98x0.95mm_HandSolder" (id 2) (at 71.628 81.915 90)
@@
   (symbol (lib_id "Device:C_Small") (at 187.96 106.045 0)
     (in_bom yes) (on_board yes) (fields_autoplaced)
-    (property "Reference" "C308" (id 0) (at 190.2841 105.1428 0)
+    (property "Reference" "C408" (id 0) (at 190.2841 105.1428 0)
       (effects (font (size 1.27 1.27)) (justify left))
     )
@@
   (symbol (lib_id "Device:Opamp_Dual") (at 132.08 92.075 0)
     (in_bom yes) (on_board yes) (fields_autoplaced)
-    (property "Reference" "U301" (id 0) (at 132.08 83.0285 0))
+    (property "Reference" "U401" (id 0) (at 132.08 83.0285 0))
     (property "Value" "lmc6042" (id 1) (at 132.08 85.8036 0))
     (property "Footprint" "Package_SO:SOIC-8_3.9x4.9mm_P1.27mm" (id 2) (at 132.08 92.075 0)
@@
   (symbol (lib_id "Device:R") (at 214.63 106.045 90)
     (in_bom yes) (on_board yes)
-    (property "Reference" "R309" (id 0) (at 209.55 104.775 90))
+    (property "Reference" "R409" (id 0) (at 209.55 104.775 90))
     (property "Value" "21k" (id 1) (at 219.075 104.775 90))
     (property "Footprint" "Resistor_SMD:R_0603_1608Metric_Pad0.98x0.95mm_HandSolder" (id 2) (at 214.63 107.823 90)
@@
   (symbol (lib_id "Device:C_Small") (at 51.435 170.18 0)
     (in_bom yes) (on_board yes) (fields_autoplaced)
-    (property "Reference" "C302" (id 0) (at 53.7591 169.2778 0)
+    (property "Reference" "C402" (id 0) (at 53.7591 169.2778 0)
       (effects (font (size 1.27 1.27)) (justify left))
     )
@@
   (symbol (lib_id "Device:C_Small") (at 59.69 111.125 270)
     (in_bom yes) (on_board yes) (fields_autoplaced)
-    (property "Reference" "C303" (id 0) (at 59.6836 105.5964 90))
+    (property "Reference" "C403" (id 0) (at 59.6836 105.5964 90))
     (property "Value" "1n8" (id 1) (at 59.6836 108.3715 90))
     (property "Footprint" "Capacitor_SMD:C_0603_1608Metric_Pad1.08x0.95mm_HandSolder" (id 2) (at 59.69 111.125 0)

Commit message: some pcb digital moved
Parts:
- C308: renamed from C408; value 100n -> 100p
- renumbered C401 to C301, C402 to C302, C403 to C303, C404 to C304, C405 to C305, C406 to C306, C407 to C307, FB401 to FB301, J401 to J301, R401 to R301, R402 to R302, R403 to R303, R404 to R304, R405 to R305, R406 to R306, R407 to R307, R408 to R308, R409 to R309, R410 to R310, U401 to U301
Other:
- note added: "cutoff at ~160kHz, do not expect the piezo to be much faster than that.. however might be unstable cus high C wurworth looking into"
- note removed: "cutoff at ~160Hz, do not expect the piezo to be much faster than that"
Changed lines of the file:
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@@
     (effects (font (size 1.27 1.27)) (justify left bottom))
   )
-  (text "cutoff at ~160Hz, do not expect the \npiezo to be much faster than that"
-    (at 154.94 87.63 0)
+  (text "cutoff at ~160kHz, do not expect the \npiezo to be much faster than that..\nhowever might be unstable cus high C wurworth looking into\n"
+    (at 140.97 86.995 0)
     (effects (font (size 1.27 1.27)) (justify left bottom))
   )
@@
   (symbol (lib_id "Device:C_Small") (at 43.18 170.18 0)
     (in_bom yes) (on_board yes)
-    (property "Reference" "C401" (id 0) (at 45.72 169.545 0)
+    (property "Reference" "C301" (id 0) (at 45.72 169.545 0)
       (effects (font (size 1.27 1.27)) (justify left))
     )
@@
   (symbol (lib_id "Device:R") (at 44.45 94.615 90)
     (in_bom yes) (on_board yes)
-    (property "Reference" "R402" (id 0) (at 38.735 93.345 90))
+    (property "Reference" "R302" (id 0) (at 38.735 93.345 90))
     (property "Value" "5k49" (id 1) (at 50.165 93.345 90))
     (property "Footprint" "Resistor_SMD:R_0603_1608Metric_Pad0.98x0.95mm_HandSolder" (id 2) (at 44.45 96.393 90)
@@
   (symbol (lib_id "Device:C_Small") (at 130.81 106.045 270)
     (in_bom yes) (on_board yes) (fields_autoplaced)
-    (property "Reference" "C407" (id 0) (at 130.8036 100.5164 90))
+    (property "Reference" "C307" (id 0) (at 130.8036 100.5164 90))
     (property "Value" "390p" (id 1) (at 130.8036 103.2915 90))
     (property "Footprint" "Capacitor_SMD:C_0603_1608Metric_Pad1.08x0.95mm_HandSolder" (id 2) (at 130.81 106.045 0)
@@
   (symbol (lib_id "Device:Opamp_Dual") (at 209.55 94.615 0)
     (in_bom yes) (on_board yes) (fields_autoplaced)
-    (property "Reference" "U401" (id 0) (at 209.55 85.5685 0))
+    (property "Reference" "U301" (id 0) (at 209.55 85.5685 0))
     (property "Value" "lmc6042" (id 1) (at 209.55 88.3436 0))
     (property "Footprint" "Package_SO:SOIC-8_3.9x4.9mm_P1.27mm" (id 2) (at 209.55 94.615 0)
@@
   (symbol (lib_id "Connector:Conn_Coaxial") (at 268.605 94.615 0)
     (in_bom yes) (on_board yes) (fields_autoplaced)
-    (property "Reference" "J401" (id 0) (at 271.145 93.9997 0)
+    (property "Reference" "J301" (id 0) (at 271.145 93.9997 0)
       (effects (font (size 1.27 1.27)) (justify left))
     )
@@
   (symbol (lib_id "Device:Opamp_Dual") (at 63.5 170.18 0)
     (in_bom yes) (on_board yes)
-    (property "Reference" "U401" (id 0) (at 61.595 169.2715 0)
+    (property "Reference" "U301" (id 0) (at 61.595 169.2715 0)
       (effects (font (size 1.27 1.27)) (justify left))
     )
@@
   (symbol (lib_id "Device:FerriteBead_Small") (at 67.31 161.29 90)
     (in_bom yes) (on_board yes)
-    (property "Reference" "FB401" (id 0) (at 67.2719 155.6217 90))
+    (property "Reference" "FB301" (id 0) (at 67.2719 155.6217 90))
     (property "Value" "BLM18AG102SN1D" (id 1) (at 67.2719 158.3968 90))
     (property "Footprint" "Inductor_SMD:L_0603_1608Metric_Pad1.05x0.95mm_HandSolder" (id 2) (at 67.31 163.068 90)
@@
   (symbol (lib_id "Device:R") (at 98.425 89.535 90)
     (in_bom yes) (on_board yes)
-    (property "Reference" "R404" (id 0) (at 92.71 88.265 90))
+    (property "Reference" "R304" (id 0) (at 92.71 88.265 90))
     (property "Value" "887" (id 1) (at 103.505 88.265 90))
     (property "Footprint" "Resistor_SMD:R_0603_1608Metric_Pad0.98x0.95mm_HandSolder" (id 2) (at 98.425 91.313 90)
@@
   (symbol (lib_id "Device:C_Small") (at 69.85 71.12 0)
     (in_bom yes) (on_board yes) (fields_autoplaced)
-    (property "Reference" "C405" (id 0) (at 72.1741 70.2178 0)
+    (property "Reference" "C305" (id 0) (at 72.1741 70.2178 0)
       (effects (font (size 1.27 1.27)) (justify left))
     )
@@
   (symbol (lib_id "Device:R") (at 166.37 92.075 90)
     (in_bom yes) (on_board yes)
-    (property "Reference" "R407" (id 0) (at 161.29 90.805 90))
+    (property "Reference" "R307" (id 0) (at 161.29 90.805 90))
     (property "Value" "10k" (id 1) (at 171.45 90.805 90))
     (property "Footprint" "Resistor_SMD:R_0603_1608Metric_Pad0.98x0.95mm_HandSolder" (id 2) (at 166.37 93.853 90)
@@
   (symbol (lib_id "Device:R") (at 245.11 94.615 90)
     (in_bom yes) (on_board yes)
-    (property "Reference" "R410" (id 0) (at 248.92 93.345 90))
+    (property "Reference" "R310" (id 0) (at 248.92 93.345 90))
     (property "Value" "33" (id 1) (at 240.665 93.345 90))
     (property "Footprint" "Resistor_SMD:R_0603_1608Metric_Pad0.98x0.95mm_HandSolder" (id 2) (at 245.11 96.393 90)
@@
   (symbol (lib_id "Device:C_Small") (at 116.84 81.915 0)
     (in_bom yes) (on_board yes) (fields_autoplaced)
-    (property "Reference" "C406" (id 0) (at 119.1641 81.0128 0)
+    (property "Reference" "C306" (id 0) (at 119.1641 81.0128 0)
       (effects (font (size 1.27 1.27)) (justify left))
     )
@@
   (symbol (lib_id "Device:R") (at 98.425 94.615 90)
     (in_bom yes) (on_board yes)
-    (property "Reference" "R405" (id 0) (at 92.71 93.345 90))
+    (property "Reference" "R305" (id 0) (at 92.71 93.345 90))
     (property "Value" "2k94" (id 1) (at 104.14 93.345 90))
     (property "Footprint" "Resistor_SMD:R_0603_1608Metric_Pad0.98x0.95mm_HandSolder" (id 2) (at 98.425 96.393 90)
@@
   (symbol (lib_id "Device:R") (at 130.81 111.125 90)
     (in_bom yes) (on_board yes)
-    (property "Reference" "R406" (id 0) (at 125.095 109.855 90))
+    (property "Reference" "R306" (id 0) (at 125.095 109.855 90))
     (property "Value" "4k75" (id 1) (at 135.89 109.855 90))
     (property "Footprint" "Resistor_SMD:R_0603_1608Metric_Pad0.98x0.95mm_HandSolder" (id 2) (at 130.81 112.903 90)
@@
   (symbol (lib_id "Device:C_Small") (at 61.595 81.915 0)
     (in_bom yes) (on_board yes) (fields_autoplaced)
-    (property "Reference" "C404" (id 0) (at 63.9191 81.0128 0)
+    (property "Reference" "C304" (id 0) (at 63.9191 81.0128 0)
       (effects (font (size 1.27 1.27)) (justify left))
     )
@@
   (symbol (lib_id "Device:R") (at 198.12 113.665 180)
     (in_bom yes) (on_board yes)
-    (property "Reference" "R408" (id 0) (at 196.85 119.38 90))
+    (property "Reference" "R308" (id 0) (at 196.85 119.38 90))
     (property "Value" "10k" (id 1) (at 196.85 109.22 90))
     (property "Footprint" "Resistor_SMD:R_0603_1608Metric_Pad0.98x0.95mm_HandSolder" (id 2) (at 199.898 113.665 90)
@@
   (symbol (lib_id "Device:R") (at 44.45 89.535 90)
     (in_bom yes) (on_board yes)
-    (property "Reference" "R401" (id 0) (at 38.735 88.265 90))
+    (property "Reference" "R301" (id 0) (at 38.735 88.265 90))
     (property "Value" "1k65" (id 1) (at 50.165 88.265 90))
     (property "Footprint" "Resistor_SMD:R_0603_1608Metric_Pad0.98x0.95mm_HandSolder" (id 2) (at 44.45 91.313 90)
@@
   (symbol (lib_id "Device:R") (at 69.85 81.915 180)
     (in_bom yes) (on_board yes)
-    (property "Reference" "R403" (id 0) (at 68.58 86.995 90))
+    (property "Reference" "R303" (id 0) (at 68.58 86.995 90))
     (property "Value" "1k87" (id 1) (at 68.58 76.835 90))
     (property "Footprint" "Resistor_SMD:R_0603_1608Metric_Pad0.98x0.95mm_HandSolder" (id 2) (at 71.628 81.915 90)
@@
   (symbol (lib_id "Device:C_Small") (at 187.96 106.045 0)
     (in_bom yes) (on_board yes) (fields_autoplaced)
-    (property "Reference" "C408" (id 0) (at 190.2841 105.1428 0)
-      (effects (font (size 1.27 1.27)) (justify left))
-    )
-    (property "Value" "100n" (id 1) (at 190.2841 107.9179 0)
+    (property "Reference" "C308" (id 0) (at 190.2841 105.1428 0)
+      (effects (font (size 1.27 1.27)) (justify left))
+    )
+    (property "Value" "100p" (id 1) (at 190.2841 107.9179 0)
       (effects (font (size 1.27 1.27)) (justify left))
     )
@@
   (symbol (lib_id "Device:Opamp_Dual") (at 132.08 92.075 0)
     (in_bom yes) (on_board yes) (fields_autoplaced)
-    (property "Reference" "U401" (id 0) (at 132.08 83.0285 0))
+    (property "Reference" "U301" (id 0) (at 132.08 83.0285 0))
     (property "Value" "lmc6042" (id 1) (at 132.08 85.8036 0))
     (property "Footprint" "Package_SO:SOIC-8_3.9x4.9mm_P1.27mm" (id 2) (at 132.08 92.075 0)
@@
   (symbol (lib_id "Device:R") (at 214.63 106.045 90)
     (in_bom yes) (on_board yes)
-    (property "Reference" "R409" (id 0) (at 209.55 104.775 90))
+    (property "Reference" "R309" (id 0) (at 209.55 104.775 90))
     (property "Value" "21k" (id 1) (at 219.075 104.775 90))
     (property "Footprint" "Resistor_SMD:R_0603_1608Metric_Pad0.98x0.95mm_HandSolder" (id 2) (at 214.63 107.823 90)
@@
   (symbol (lib_id "Device:C_Small") (at 51.435 170.18 0)
     (in_bom yes) (on_board yes) (fields_autoplaced)
-    (property "Reference" "C402" (id 0) (at 53.7591 169.2778 0)
+    (property "Reference" "C302" (id 0) (at 53.7591 169.2778 0)
       (effects (font (size 1.27 1.27)) (justify left))
     )
@@
   (symbol (lib_id "Device:C_Small") (at 59.69 111.125 270)
     (in_bom yes) (on_board yes) (fields_autoplaced)
-    (property "Reference" "C403" (id 0) (at 59.6836 105.5964 90))
+    (property "Reference" "C303" (id 0) (at 59.6836 105.5964 90))
     (property "Value" "1n8" (id 1) (at 59.6836 108.3715 90))
     (property "Footprint" "Capacitor_SMD:C_0603_1608Metric_Pad1.08x0.95mm_HandSolder" (id 2) (at 59.69 111.125 0)
